File: SynBioDesign-LEDPCB/SynBioDesign-LEDPCB.kicad_pcb (KiCad board)
At the start: 2 copper layers, 18 x 23 mm, 7 parts, among them J1 Conn_02x03_Odd_Even, J2 Conn_02x03_Odd_Even, J3 Conn_02x03_Odd_Even, J4 Conn_02x03_Odd_Even

Commit message: Adding silk
Other:
- board text added: "SynBioDesign LED PCB"
Changed lines of the file:
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@@
   )
   (gr_rect (start 143.5 83.5) (end 161.5 106.5) (layer "Edge.Cuts") (width 0.1) (fill none))
+  (gr_text "SynBioDesign\nLED PCB" (at 153 98) (layer "B.SilkS")
+    (effects (font (size 1.5 1.5) (thickness 0.3)) (justify mirror))
+  )
   (gr_text "B0" (at 150 100) (layer "F.SilkS")
     (effects (font (size 0.75 0.75) (thickness 0.15)))
